Commit message: Kinematics using Modern Robotics Library

File: World/models/thor_robot.urdf (robot description, URDF)
Before this commit: robot thor, 7 links, 6 joints
Links:
- link art1: geometry visual mesh filename=thor_meshes/art1.stl scale=0.001 0.001 0.001
- link art2: geometry visual mesh filename=thor_meshes/art2.stl scale=0.001 0.001 0.001
- link art3: geometry visual mesh filename=thor_meshes/art3.stl scale=0.001 0.001 0.001
- link art4: geometry visual mesh filename=thor_meshes/art4.stl scale=0.001 0.001 0.001
- link art5: geometry visual mesh filename=thor_meshes/art5.stl scale=0.001 0.001 0.001
- link art6: geometry visual mesh filename=thor_meshes/art6.stl scale=0.001 0.001 0.001
- link base: geometry visual mesh filename=thor_meshes/base.stl scale=0.001 0.001 0.001
